File: output/pcbs/speedy-o.kicad_pcb (KiCad board)
At the start: 2 copper layers, 159.3 x 108.6 mm, 93 parts

Commit message: first satisfying layout
Parts:
- removed _2, _3, _4, _5, _6: , MountingHole_2.2mm_M2_Pad_Via
- added H1: , ceoloide:mounting_hole_plated, F.Cu at (120.0, 78.0)
- added H2: , ceoloide:mounting_hole_plated, F.Cu at (134.4, 146.0)
- added H3: , ceoloide:mounting_hole_plated, F.Cu at (170.4, 146.0)
- added H4: , ceoloide:mounting_hole_plated, F.Cu at (213.1, 136.7)
- added H5: , ceoloide:mounting_hole_plated, F.Cu at (201.0, 80.0)
- LED1, LED10, LED11, LED12, LED13, LED14, LED15, LED16, LED17, LED18, LED19, LED2, LED20, LED21, LED22, LED23, LED24, LED25, LED26, LED27, LED3, LED4, LED5, LED6, LED7, LED8, LED9: footprint WS2812B -> ceoloide:led_SK6812mini-e (per-key, reversible); moved to B.Cu
Connections:
- D1 pad 1: P6 -> P16
- D2 pad 1: P7 -> P6
- D3 pad 1: P8 -> P7
- D4 pad 1: P9 -> P8
- LED1 pad 2: rgb_main_outer_home -> rgb_main_outer_bottom
- LED1 pad 4: rgb_main_outer_bottom -> rgb_main_outer_home
- LED10 pad 2: rgb_main_pinky_top -> rgb_main_ring_home
- LED10 pad 4: rgb_main_ring_home -> rgb_main_pinky_top
- LED11 pad 2: rgb_main_middle_top -> rgb_main_ring_top
- LED11 pad 4: rgb_main_ring_top -> rgb_main_middle_top
- LED12 pad 2: (no net) -> rgb_main_ring_num
- LED12 pad 4: rgb_main_ring_num -> (no net)
- LED13 pad 2: rgb_main_index_bottom -> rgb_main_middle_bottom
- LED13 pad 4: rgb_main_middle_bottom -> rgb_main_index_bottom
- LED14 pad 2: rgb_main_ring_home -> rgb_main_middle_home
- LED14 pad 4: rgb_main_middle_home -> rgb_main_ring_home
- LED15 pad 2: rgb_main_index_top -> rgb_main_middle_top
- LED15 pad 4: rgb_main_middle_top -> rgb_main_index_top
- LED16 pad 2: rgb_main_ring_num -> rgb_main_middle_num
- LED16 pad 4: rgb_main_middle_num -> rgb_main_ring_num
- LED17 pad 2: rgb_main_inner_bottom -> rgb_main_index_bottom
- LED17 pad 4: rgb_main_index_bottom -> rgb_main_inner_bottom
- LED18 pad 2: rgb_main_middle_home -> rgb_main_index_home
- LED18 pad 4: rgb_main_index_home -> rgb_main_middle_home
- LED19 pad 2: rgb_main_inner_top -> rgb_main_index_top
- LED19 pad 4: rgb_main_index_top -> rgb_main_inner_top
- LED2 pad 2: rgb_main_pinky_home -> rgb_main_outer_home
- LED2 pad 4: rgb_main_outer_home -> rgb_main_pinky_home
- LED20 pad 2: rgb_main_middle_num -> rgb_main_index_num
- LED20 pad 4: rgb_main_index_num -> rgb_main_middle_num
- LED21 pad 2: rgb_main_inner_home -> rgb_main_inner_bottom
- LED21 pad 4: rgb_main_inner_bottom -> rgb_main_inner_home
- LED22 pad 2: rgb_main_index_home -> rgb_main_inner_home
- LED22 pad 4: rgb_main_inner_home -> rgb_main_index_home
- LED23 pad 2: rgb_main_inner_num -> rgb_main_inner_top
- LED23 pad 4: rgb_main_inner_top -> rgb_main_inner_num
- LED24 pad 2: rgb_main_index_num -> rgb_main_inner_num
- LED24 pad 4: rgb_main_inner_num -> rgb_main_index_num
- LED25 pad 2: rgb_main_pinky_bottom -> rgb_thumb_outer_home
- LED25 pad 4: rgb_thumb_outer_home -> rgb_main_pinky_bottom
- LED26 pad 2: rgb_thumb_outer_home -> rgb_thumb_home_home
- LED26 pad 4: rgb_thumb_home_home -> rgb_thumb_outer_home
- LED27 pad 2: rgb_thumb_home_home -> P19
- LED27 pad 4: P9 -> rgb_thumb_home_home
- LED3 pad 2: rgb_main_outer_num -> rgb_main_outer_top
- LED3 pad 4: rgb_main_outer_top -> rgb_main_outer_num
- LED4 pad 2: rgb_main_pinky_num -> rgb_main_outer_num
- LED4 pad 4: rgb_main_outer_num -> rgb_main_pinky_num
- LED5 pad 2: rgb_main_outer_bottom -> rgb_main_pinky_bottom
- LED5 pad 4: rgb_main_pinky_bottom -> rgb_main_outer_bottom
- LED6 pad 2: rgb_main_ring_bottom -> rgb_main_pinky_home
- LED6 pad 4: rgb_main_pinky_home -> rgb_main_ring_bottom
- LED7 pad 2: rgb_main_outer_top -> rgb_main_pinky_top
- LED7 pad 4: rgb_main_pinky_top -> rgb_main_outer_top
- LED8 pad 2: rgb_main_ring_top -> rgb_main_pinky_num
- LED8 pad 4: rgb_main_pinky_num -> rgb_main_ring_top
- LED9 pad 2: rgb_main_middle_bottom -> rgb_main_ring_bottom
- LED9 pad 4: rgb_main_ring_bottom -> rgb_main_middle_bottom
Routing:
- net VCC: track 0.00 -> 101.4 mm, vias 0 -> 27
- net GND: track 0.00 -> 101.4 mm, vias 0 -> 27
- net rgb_thumb_outer_home: track 0.00 -> 13.5 mm, vias 0 -> 2
- net rgb_thumb_home_home: track 0.00 -> 13.5 mm, vias 0 -> 2
- net rgb_main_middle_bottom: track 0.00 -> 13.5 mm, vias 0 -> 2
- net rgb_main_inner_bottom: track 0.00 -> 13.5 mm, vias 0 -> 2
- net rgb_main_index_bottom: track 0.00 -> 13.5 mm, vias 0 -> 2
- net rgb_main_inner_home: track 0.00 -> 13.5 mm, vias 0 -> 2
- net rgb_main_ring_num: track 0.00 -> 13.5 mm, vias 0 -> 2
- net rgb_main_ring_home: track 0.00 -> 13.5 mm, vias 0 -> 2
- net rgb_main_middle_top: track 0.00 -> 13.5 mm, vias 0 -> 2
- net rgb_main_middle_num: track 0.00 -> 13.5 mm, vias 0 -> 2
- net rgb_main_middle_home: track 0.00 -> 13.5 mm, vias 0 -> 2
- net rgb_main_inner_top: track 0.00 -> 13.5 mm, vias 0 -> 2
- net rgb_main_inner_num: track 0.00 -> 13.5 mm, vias 0 -> 2
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Other:
- net class Default removed
